Commit message: esemplified urdf in lesson 5

File: L5-Digital-Twin-with-URDF/arduinobot_ws/src/arduinobot_description/urdf/arduinobot.urdf.xacro (robot description, xacro)
@@ -162,51 +162,3 @@
         <origin xyz="0 0 0"/>
     </joint>
-    <!-- Transmissions-->
-    <transmission name="transmission_1">
-        <type>transmission_interface/SimpleTransmission</type>
-        <joint name="joint_1">
-            <hardwareInterface>PositionJointInterface</hardwareInterface>
-        </joint>
-        <actuator name="motor_1">
-            <hardwareInterface>PositionJointInterface</hardwareInterface>
-            <mechanicalReduction>1</mechanicalReduction>
-        </actuator>
-    </transmission>
-    <transmission name="transmission_2">
-        <type>transmission_interface/SimpleTransmission</type>
-        <joint name="joint_2">
-            <hardwareInterface>PositionJointInterface</hardwareInterface>
-        </joint>
-        <actuator name="motor_2">
-            <hardwareInterface>PositionJointInterface</hardwareInterface>
-            <mechanicalReduction>1</mechanicalReduction>
-        </actuator>
-    </transmission>
-    <transmission name="transmission_3">
-        <type>transmission_interface/SimpleTransmission</type>
-        <joint name="joint_3">
-            <hardwareInterface>PositionJointInterface</hardwareInterface>
-        </joint>
-        <actuator name="motor_3">
-            <hardwareInterface>PositionJointInterface</hardwareInterface>
-            <mechanicalReduction>1</mechanicalReduction>
-        </actuator>
-    </transmission>
-    <transmission name="transmission_4">
-        <type>transmission_interface/SimpleTransmission</type>
-        <joint name="joint_4">
-            <hardwareInterface>PositionJointInterface</hardwareInterface>
-        </joint>
-        <actuator name="motor_4">
-            <hardwareInterface>PositionJointInterface</hardwareInterface>
-            <mechanicalReduction>1</mechanicalReduction>
-        </actuator>
-    </transmission>
-    <!-- Gazebo Configuration section -->
-    <gazebo>
-        <plugin name="gazebo_ros_control" filename="libgazebo_ros_control.so">
-            <robotNamespace>/arduinobot</robotNamespace>
-            <robotSimType>gazbo_roscontrol/DefaultRobotHWSim</robotSimType>
-        </plugin>
-    </gazebo>
 </robot>

Commit message: small change to the urdf file

File: L5-Digital-Twin-with-URDF/arduinobot_ws/src/arduinobot_description/urdf/arduinobot.urdf.xacro (robot description, xacro)
@@ -10,5 +10,4 @@
     <xacro:property name="up_limit_horizontal_arm_arm_rotation" value="${PI/2}" />
     <!-- Links -->
-    <link name="world"/>
     <link name="base_link">
         <visual>
@@ -111,9 +110,4 @@
     <link name="tool_link"></link>
     <!-- Joints -->
-    <joint name="joint_world" type="fixed">
-        <parent link="world" />
-        <child link="base_link" />
-        <origin xyz="0 0 0" rpy="0 0 0" />
-    </joint>
     <joint name ="joint_1" type="revolute">
         <parent link="base_link"/>

Commit message: added documentation up to the Lesson 5

File: L5-Digital-Twin-with-URDF/arduinobot_ws/src/arduinobot_description/urdf/arduinobot.urdf.xacro (robot description, xacro)
@@ -3,12 +3,18 @@
     <!-- Useful Variables (Properties) -->
     <xacro:property name="PI" value="3.14159265359" />
-    <xacro:property name="low_limit_base_plate_rotation" value="-${PI/2}" />
-    <xacro:property name="up_limit_base_plate_rotation" value="${PI/2}" />
-    <xacro:property name="low_limit_forward_drive_arm_rotation" value="-${PI/2}" />
-    <xacro:property name="up_limit_forward_drive_arm_rotation" value="${PI/2}" />
-    <xacro:property name="low_limit_horizontal_arm_rotation" value="-${PI/2}" />
-    <xacro:property name="up_limit_horizontal_arm_arm_rotation" value="${PI/2}" />
     <!-- Links -->
+    <link name="world"/>
+    <joint name="virtual_joint" type="fixed">
+        <parent link="world"/>
+        <child link="base_link"/>
+        <origin xyz="0 0 0.25"/>
+    </joint>
     <link name="base_link">
+        <inertial>
+                <mass value="1" />
+                <inertia ixx="1.0" ixy="0.0" ixz="0.0"
+                     iyy="1.0" iyz="0.0"
+                     izz="1.0" />
+        </inertial>
         <visual>
             <origin rpy="0 0 0" xyz="-0.5 -0.5 0"/>
@@ -25,4 +31,10 @@
     </link>
     <link name="base_plate">
+        <inertial>
+                <mass value="0.1" />
+                <inertia ixx="1.0" ixy="0.0" ixz="0.0"
+                     iyy="1.0" iyz="0.0"
+                     izz="1.0" />
+        </inertial>
         <visual>
             <origin rpy="0 0 0" xyz="-0.39 -0.39 -0.56"/>
@@ -39,4 +51,10 @@
     </link>
     <link name="forward_drive_arm">
+        <inertial>
+                <mass value="0.1" />
+                <inertia ixx="1.0" ixy="0.0" ixz="0.0"
+                     iyy="1.0" iyz="0.0"
+                     izz="1.0" />
+        </inertial>
         <visual>
             <origin rpy=" 0 -${PI/2} ${PI/2}" xyz="0.19 0.06 -0.08"/>
@@ -53,4 +71,10 @@
     </link>
     <link name="horizontal_arm">
+        <inertial>
+                <mass value="0.1" />
+                <inertia ixx="1.0" ixy="0.0" ixz="0.0"
+                     iyy="1.0" iyz="0.0"
+                     izz="1.0" />
+        </inertial>
         <visual>
             <origin rpy="${PI/2} 0 ${PI/2}" xyz="-0.03 -0.4 -0.06"/>
@@ -67,4 +91,10 @@
     </link>
     <link name="claw_support">
+        <inertial>
+                <mass value="0.05" />
+                <inertia ixx="1.0" ixy="0.0" ixz="0.0"
+                     iyy="1.0" iyz="0.0"
+                     izz="1.0" />
+        </inertial>
         <visual>
             <origin rpy="0 0 ${PI/2}" xyz="0 -0.05 -0.15"/>
@@ -81,4 +111,10 @@
     </link>
     <link name="gripper_right">
+        <inertial>
+                <mass value="0.01" />
+                <inertia ixx="1.0" ixy="0.0" ixz="0.0"
+                     iyy="1.0" iyz="0.0"
+                     izz="1.0" />
+        </inertial>
         <visual>
             <origin rpy="0 0 -${PI/2}" xyz="-0.1 0.50 -0.1"/>
@@ -95,4 +131,10 @@
     </link>
     <link name="gripper_left">
+        <inertial>
+                <mass value="0.01" />
+                <inertia ixx="1.0" ixy="0.0" ixz="0.0"
+                     iyy="1.0" iyz="0.0"
+                     izz="1.0" />
+        </inertial>
         <visual>
             <origin rpy="0 0 -${PI/2}" xyz="-0.04 0.50 -0.1"/>
@@ -102,5 +144,5 @@
         </visual>
         <collision>
-            <origin rpy="0 0 -${PI/2}" xyz="-0.2 0.50 -0.1"/>
+            <origin rpy="0 0 -${PI/2}" xyz="-0.04 0.50 -0.1"/>
             <geometry>
                 <mesh filename="package://arduinobot_description/mesh/left_finger.STL" scale="0.01 0.01 0.01"/>
@@ -115,12 +157,12 @@
         <origin xyz="0 0 0.307"/>
         <axis xyz="0 0 1"/>
-        <limit lower="-${PI/2}" upper="${PI/2}" effort="1000.0" velocity="0.5"/>
+        <limit lower="-${PI/2}" upper="${PI/2}" effort="30.0" velocity="0.5"/>
     </joint>
     <joint name ="joint_2" type="revolute">
         <parent link="base_plate"/>
         <child link = "forward_drive_arm"/>
-        <origin xyz="0 0 0.28"/>
+        <origin xyz="-0.02 0 0.35"/>
         <axis xyz="1 0 0"/>
-        <limit lower="-${PI/2}" upper="${PI/2}" effort="1000.0" velocity="0.5"/>
+        <limit lower="-${PI/2}" upper="${PI/2}" effort="30.0" velocity="0.5"/>
     </joint>
     <joint name ="joint_3" type="revolute">
@@ -129,5 +171,5 @@
         <origin xyz="0 0 0.8"/>
         <axis xyz="1 0 0"/>
-        <limit lower="-${PI/2}" upper="${PI/2}" effort="1000.0" velocity="0.5"/>
+        <limit lower="-${PI/2}" upper="${PI/2}" effort="30.0" velocity="0.5"/>
     </joint>
     <joint name ="horizontal_arm_to_claw_support" type="fixed">
@@ -141,5 +183,5 @@
         <origin xyz="-0.04 0.13 -0.1"/>
         <axis xyz="0 0 1"/>
-        <limit lower="-${PI/2}" upper="0" effort="1000.0" velocity="0.5"/>
+        <limit lower="-${PI/2}" upper="0" effort="30.0" velocity="0.5"/>
     </joint>
     <joint name ="joint_5" type="revolute">
@@ -148,5 +190,5 @@
         <origin xyz="-0.22 0.13 -0.1"/>
         <axis xyz="0 0 1"/>
-        <limit lower="0" upper="${PI/2}" effort="1000.0" velocity="0.5"/>
+        <limit lower="0" upper="${PI/2}" effort="30.0" velocity="0.5"/>
         <mimic joint="joint_4" multiplier="-1" offset="0"/>
     </joint>
@@ -156,3 +198,62 @@
         <origin xyz="0 0 0"/>
     </joint>
+    <!-- Transmissions-->
+    <transmission name="transmission_1">
+        <type>transmission_interface/SimpleTransmission</type>
+        <joint name="joint_1">
+            <hardwareInterface>hardware_interface/PositionJointInterface</hardwareInterface>
+        </joint>
+        <actuator name="motor_1">
+            <hardwareInterface>hardware_interface/PositionJointInterface</hardwareInterface>
+            <mechanicalReduction>1</mechanicalReduction>
+        </actuator>
+    </transmission>
+    <transmission name="transmission_2">
+        <type>transmission_interface/SimpleTransmission</type>
+        <joint name="joint_2">
+            <hardwareInterface>hardware_interface/PositionJointInterface</hardwareInterface>
+        </joint>
+        <actuator name="motor_2">
+            <hardwareInterface>hardware_interface/PositionJointInterface</hardwareInterface>
+            <mechanicalReduction>1</mechanicalReduction>
+        </actuator>
+    </transmission>
+    <transmission name="transmission_3">
+        <type>transmission_interface/SimpleTransmission</type>
+        <joint name="joint_3">
+            <hardwareInterface>hardware_interface/PositionJointInterface</hardwareInterface>
+        </joint>
+        <actuator name="motor_3">
+            <hardwareInterface>hardware_interface/PositionJointInterface</hardwareInterface>
+            <mechanicalReduction>1</mechanicalReduction>
+        </actuator>
+    </transmission>
+    <transmission name="transmission_4">
+        <type>transmission_interface/SimpleTransmission</type>
+        <joint name="joint_4">
+            <hardwareInterface>hardware_interface/PositionJointInterface</hardwareInterface>
+        </joint>
+        <actuator name="motor_4">
+            <hardwareInterface>hardware_interface/PositionJointInterface</hardwareInterface>
+            <mechanicalReduction>1</mechanicalReduction>
+        </actuator>
+    </transmission>
+    <transmission name="transmission_5">
+        <type>transmission_interface/SimpleTransmission</type>
+        <joint name="joint_5">
+            <hardwareInterface>hardware_interface/PositionJointInterface</hardwareInterface>
+        </joint>
+        <actuator name="motor_5">
+            <hardwareInterface>hardware_interface/PositionJointInterface</hardwareInterface>
+            <mechanicalReduction>1</mechanicalReduction>
+        </actuator>
+    </transmission>
+    <!-- ros_control plugin -->
+    <gazebo>
+        <plugin name="gazebo_ros_control" filename="libgazebo_ros_control.so">
+            <robotNamespace>/arduinobot_sim</robotNamespace>
+            <robotSimType>gazebo_ros_control/DefaultRobotHWSim</robotSimType>
+            <legacyModeNS>true</legacyModeNS>
+        </plugin>
+    </gazebo>
 </robot>
